File: circuit/projects/controller/controllerv6.kicad_sch (KiCad schematic)
At the start: 51 parts, among them J1 Conn_01x02, SW1 SW_DIP_x01, SW10 SW_DIP_x01, SW2 SW_DIP_x01, SW3 SW_DIP_x01, SW4 SW_DIP_x01, SW5 SW_DIP_x01, SW6 SW_DIP_x01, SW7 SW_DIP_x01, SW8 TOGGLE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

Commit message: ピン番号の更新と回路データの更新
Parts:
- added R19: 10k, Resistor_THT:R_Axial_DIN0204_L3.6mm_D1.6mm_P7.62mm_Horizontal, symbol Device:R
- added SW11: TOGGLE, Connector_PinHeader_2.54mm:PinHeader_1x03_P2.54mm_Vertical, symbol s-ken:TOGGLE
- C1: value 10μ -> 0.1μ
- C2: value 0.1μ -> 10μ; footprint Capacitor_THT:C_Disc_D3.0mm_W1.6mm_P2.50mm -> Capacitor_THT:CP_Radial_Tantal_D6.0mm_P2.50mm
- C4, C5: footprint Capacitor_THT:C_Disc_D3.0mm_W1.6mm_P2.50mm -> Capacitor_THT:CP_Radial_Tantal_D6.0mm_P2.50mm
- J1: footprint Connector_AMASS:AMASS_XT30PW-M_1x02_P2.50mm_Horizontal -> Connector_AMASS:AMASS_XT30PW-F_1x02_P2.50mm_Horizontal
Connections:
- net +3.3V: now also R19.2
- net +BATT: now also J1.2 (Pin_2); no longer J1.1 (Pin_1)
- net BUSY: no longer U2.36 (22/GPIO22)
- net GND: now also J1.1 (Pin_1), SW11.2 (P); no longer J1.2 (Pin_2)
- net IM920RX: now also U2.37 (23/GPIO23); no longer U2.35 (TX/UOTXD)
- net IM920TX: now also U2.36 (22/GPIO22); no longer U2.34 (RX/UORXD)
- net RESET: no longer U2.37 (23/GPIO23)
- net sw5: now also U2.28 (17/GPIO17); no longer U2.23 (15/GPIO15/MTDO)
- net sw6: now also U2.30 (18/GPIO18); no longer U2.25 (0/GPIO0)
- net sw7: now also U2.29 (5/GPIO5); no longer U2.24 (2/GPIO2)
- net sw8: now also U2.31 (19/GPIO19); no longer U2.26 (4/GPIO4)
- net sw11: now reaches U2.33 (21/GPIO21)
- net sw11: now also R19.1, SW11.1 (O)
Other:
- moved on the sheet: J1
